File: KiCad/CCD-Arduino-Mega.kicad_pcb (KiCad board)
At the start: 2 copper layers, 105.4 x 53.3 mm, 36 parts, among them J1 CCD+, J10 +5V, J11 PWM, J12 PWM, J13 COMMUNICATION, J2 CCD-, J3 Ground, J4 CCD-BUS, J5 Button, J6 POWER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

Commit message: implement ZIF-Socket
Parts:
- U1: footprint Package_DIP:DIP-14_W7.62mm -> Socket:DIP_Socket-14_W4.3_W5.08_W7.62_W10.16_W10.9_3M_214-3339-00-0602J
- moved J5 15.5 mm to (107.7, 102.9), turned to 90 degrees
- moved U1 15.3 mm to (154.9, 101.6), turned to -90 degrees
- moved R4 14.2 mm to (113.0, 96.5), turned to 90 degrees
- moved JP4 12.7 mm to (124.5, 94.0), turned to -90 degrees
- moved R5 2.84 mm to (124.5, 121.9)
- moved R8 2.54 mm to (124.5, 83.8)
- moved R9 2.54 mm to (124.5, 88.9)
- moved X1 2.54 mm to (116.8, 101.6)
Routing:
- net /CLK: track 38.4 -> 54.9 mm
- net /CONTROL: track 47.6 -> 60.6 mm
- net /D2: track 45.8 -> 58.1 mm
- net /TX1: track 50.9 -> 63.2 mm
- net /REC: track 55.2 -> 65.5 mm
- net /Button: track 58.7 -> 50.6 mm
- net /BUS-: track 31.5 -> 38.0 mm
- net /BUS+: track 30.5 -> 36.3 mm
- net Net-(JP4-Pad2): track 13.8 -> 8.67 mm
- net Net-(D1-Pad2): track 7.41 -> 4.87 mm
- net /D13: track 7.40 -> 9.20 mm
- net Net-(D2-Pad2): track 16.1 -> 14.3 mm
- net /CCD-: track 60.7 -> 62.5 mm
- net /D12: track 12.8 -> 13.8 mm
