File: KiCad/CCD-Arduino-Mega.kicad_pcb (KiCad board)
At the start: 2 copper layers, 105.4 x 53.3 mm, 36 parts, among them J1 CCD+, J10 +5V, J11 PWM, J12 PWM, J13 COMMUNICATION, J2 CCD-, J3 Ground, J4 CCD-BUS, J5 Button, J6 POWER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

Commit message: remove LED, connect CLK; Revision 1.0
Parts:
- removed D2: LED, LED_THT:LED_D5.0mm
- removed R9: 220Ω, Resistor_THT:R_Axial_DIN0207_L6.3mm_D2.5mm_P7.62mm_Horizontal
- added REF**: OSHW-Logo2_14.6x12mm_SilkScreen, Symbol:OSHW-Logo2_14.6x12mm_SilkScreen, F.Cu at (142.2, 88.9)
- J3, TP3: value Ground -> GND
- JP1: value Termination -> TERMINATION
- JP4: value Jumper_NC_Dual -> Quarz_Enable
- U1: value Conn_02x07_Counter_Clockwise -> CCD-Interface
- moved R4 12.5 mm to (124.5, 91.4), turned to 180 degrees
- moved JP4 5.67 mm to (119.4, 96.5), turned to 90 degrees
- moved D1 3.80 mm to (106.7, 81.3)
- moved R8 2.54 mm to (124.5, 86.4)
- moved J5 1.30 mm to (108.0, 101.6)
- moved SW1 0.77 mm to (110.5, 109.2)
Connections:
- J11 pad 6: /D12 -> /Button
- J11 pad 7: /Button -> /CLK
Routing:
- net /CLK: track 54.9 -> 97.5 mm
- net (no net): track 16.5 -> 0.00 mm
- net Net-(D2-Pad2): track 14.3 -> 0.00 mm
- net /D12: track 13.8 -> 0.00 mm
- net Net-(D1-Pad2): track 4.87 -> 9.72 mm
- net Net-(JP4-Pad2): track 8.67 -> 6.14 mm
- net /Button: track 50.6 -> 48.7 mm
- net /D13: track 9.20 -> 10.3 mm
Other:
- board text added: "CCD-Arduino-Mega Rev1.0 github.com/Moddler © Moddler 2022"
