File: KiCad/CCD-Arduino-Mega.kicad_pcb (KiCad board)
At the start: 2 copper layers, 105.4 x 53.3 mm, 35 parts, among them J1 CCD+, J10 +5V, J11 PWM, J12 PWM, J13 COMMUNICATION, J2 CCD-, J3 GND, J4 CCD-BUS, J5 Button, J6 POWER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

Commit message: Add "ZIF" to PCB
Other:
- board text added: "CCD-Arduino-Mega Rev1.0 ZIF github.com/Moddler © Moddler 2022"
- board text removed: "CCD-Arduino-Mega Rev1.0 github.com/Moddler © Moddler 2022"
Changed lines of the file:
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@@
   (gr_line (start 200.66 99.06) (end 207.01 93.98) (layer "Edge.Cuts") (width 0.05))
   (gr_circle (center 191.77 78.74) (end 193.3575 78.74) (layer "Edge.Cuts") (width 0.15) (fill none))
-  (gr_text "CCD-Arduino-Mega Rev1.0\ngithub.com/Moddler\n© Moddler 2022" (at 149 119.38) (layer "F.SilkS")
+  (gr_text "CCD-Arduino-Mega Rev1.0 ZIF\ngithub.com/Moddler\n© Moddler 2022" (at 149 119.38) (layer "F.SilkS")
     (effects (font (size 1.5 1.5) (thickness 0.3)))
   )

Commit message: correction R value
Parts:
- R1: value 120kΩ -> 120Ω
Changed lines of the file:
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@@
       (effects (font (size 1 1) (thickness 0.15)))
     )
-    (fp_text value "120kΩ" (at 3.81 2.37 90) (layer "F.Fab")
+    (fp_text value "120Ω" (at 3.81 2.37 90) (layer "F.Fab")
       (effects (font (size 1 1) (thickness 0.15)))
     )
